Commit message: Continued work on bringing sensors over

File: install/husky_description/share/husky_description/urdf/accessories/intel_realsense.urdf.xacro (robot description, xacro)
@@ -33,5 +33,5 @@
               <width>${width}</width>
               <height>${height}</height>
-              <!-- TODO: check what format the Realsense hardware delivers and set this to match! -->
+              <!-- check what format the Realsense hardware delivers and set this to match! -->
               <format>RGB8</format>
             </image>

File: install/husky_description/share/husky_description/urdf/husky_macro.urdf.xacro (robot description, xacro)
@@ -24,5 +24,5 @@
   <xacro:arg name="laser_3d_xyz" default="$(optenv HUSKY_LASER_3D_XYZ 0 0 0)" />
   <xacro:arg name="laser_3d_rpy" default="$(optenv HUSKY_LASER_3D_RPY 0 0 0)" />
-  <xacro:arg name="realsense_enabled" default="$(optenv HUSKY_REALSENSE_ENABLED false)" />
+  <xacro:arg name="realsense_enabled" default="$(optenv HUSKY_REALSENSE_ENABLED 1)" />
   <xacro:arg name="realsense_xyz" default="$(optenv HUSKY_REALSENSE_XYZ 0 0 0)" />
   <xacro:arg name="realsense_rpy" default="$(optenv HUSKY_REALSENSE_RPY 0 0 0)" />
@@ -171,5 +171,5 @@
   <xacro:property name="sensorbar_needed_lidar"     value="$(arg laser_3d_enabled)" />
   <xacro:property name="sensorbar_needed_zed2" value="$(arg zed2_enabled)" />
-  <xacro:if value="true">
+  <xacro:if value="$(arg sensor_arch)">
     <xacro:sensor_arch prefix="" parent="top_plate_link" size="$(arg sensor_arch_height)">
         <origin xyz="$(optenv HUSKY_SENSOR_ARCH_OFFSET 0 0 0.5)" rpy="$(optenv HUSKY_SENSOR_ARCH_RPY 0 0 0)"/>
@@ -186,4 +186,14 @@
       <xacro:intel_realsense_mount prefix="camera" topic="realsense" parent_link="realsense_mountpoint"/>
     </xacro:if>
+  <!-- Custom addition to xacro file to include ZED2 camera ; by Dev Vaibhav-->
+  <!-- add the zed2 to the sensor arch if needed -->
+  <xacro:if value="$(arg zed2_enabled)">
+    <link name="zed2_mountpoint"/>
+    <joint name="zed2_mountpoint_joint" type="fixed">
+      <origin xyz="$(arg zed2_xyz)" rpy="$(arg zed2_rpy)" />
+      <parent link="$(arg zed2_mount)"/>
+      <child link="zed2_mountpoint" />
+    </joint>
+  </xacro:if>
     <ros2_control name="${prefix}husky_hardware" type="system">
       <hardware>

Commit message: Added standin STL for realsense, removed inertia component from arch and fixed coordinate frame

File: install/husky_description/share/husky_description/urdf/accessories/intel_realsense.urdf.xacro (robot description, xacro)
@@ -78,5 +78,5 @@
         <geometry>
           <!-- Origin of this mesh is the base of the bracket. -->
-          <mesh filename="package://realsense2_description/meshes/d415.stl" />
+          <mesh filename="file://$(find husky_description)/meshes/accessories/realsense.stl" />
         </geometry>
         <material name="white" />

File: install/husky_description/share/husky_description/urdf/accessories/sensor_arch.urdf.xacro (robot description, xacro)
@@ -3,5 +3,5 @@
   <xacro:macro name="sensor_arch" params="prefix parent size:=510 *origin">
       <!-- Robot Base -->
-      <xacro:macro name="box_inertia" params="m w h d">
+      <!--xacro:macro name="box_inertia" params="m w h d">
         <inertial>
           <origin xyz="0 0 0" rpy="0 0 0"/>
@@ -9,5 +9,6 @@
           <inertia ixx="${(m/12) * (h*h + d*d)}" ixy="0.0" ixz="0.0" iyy="${(m/12) * (w*w + d*d)}" iyz="0.0" izz="${(m/12) * (w*w + h*h)}"/>
         </inertial>
-      </xacro:macro>
+      </xacro:macro>-->
+  <link name="${prefix}sensor_arch_base_link" />
   <link name="${prefix}sensor_arch_mount_link">
      <origin xyz="0 0 0" rpy="0 0 0"/>
@@ -23,11 +24,17 @@
         </geometry>
     </collision>
-    <xacro:box_inertia m=".01" w=".01" d=".01" h=".01"/>
+    <!--<xacro:box_inertia m=".01" w=".01" d=".01" h=".01"/>-->
   </link>
-  <joint name="${prefix}sensor_arch_mount" type="fixed">
-  	    <xacro:insert_block name="origin" />
+  <joint name="${prefix}sensor_arch_base_link_joint" type="fixed">
             <parent link="${parent}" />
-            <child link="${prefix}sensor_arch_mount_link" />
-  </joint>
+            <child link="${prefix}sensor_arch_base_link" />
+            <xacro:insert_block name="origin" />
+        </joint>
+        <!-- Attach the sensor arch to the top plate -->
+        <joint name="${prefix}sensor_arch_mount" type="fixed">
+             <parent link="${prefix}sensor_arch_base_link"/>
+             <child link="${prefix}sensor_arch_mount_link"/>
+             <origin xyz="0 0 ${size/1000}" rpy="0 0 0" />
+        </joint>
 </xacro:macro>
 </robot>

File: install/husky_description/share/husky_description/urdf/husky_macro.urdf.xacro (robot description, xacro)
@@ -1,13 +1,13 @@
 <?xml version="1.0"?>
-<robot xmlns:xacro="http://ros.org/wiki/xacro">
-<!-- lms1xx_xyz broked :(
-  <xacro:arg name="laser_enabled" default="false" />
+<robot name="husky" xmlns:xacro="http://ros.org/wiki/xacro">
+  <!-- lms1xx_xyz broken :(
+  <xacro:arg name="laser_enabled" default="$(optenv HUSKY_LMS1XX_ENABLED 0)" />
   <xacro:arg name="laser_xyz" default="$(optenv HUSKY_LMS1XX_XYZ 0.2206 0.0 0.00635)" />
   <xacro:arg name="laser_rpy" default="$(optenv HUSKY_LMS1XX_RPY 0.0 0.0 0.0)" />
-  <xacro:arg name="laser_secondary_enabled" default="false" />
+  <xacro:arg name="laser_secondary_enabled" default="$(optenv HUSKY_LMS1XX_SECONDARY_ENABLED 0)" />
   <xacro:arg name="laser_secondary_xyz" default="$(optenv HUSKY_LMS1XX_SECONDARY_XYZ -0.2206 0.0 0.00635)" />
   <xacro:arg name="laser_secondary_rpy" default="$(optenv HUSKY_LMS1XX_SECONDARY_RPY 0.0 0.0 3.14159)" />
 -->
-  <xacro:arg name="laser_ust10_front_enabled" default="false" />
+  <xacro:arg name="laser_ust10_front_enabled" default="$(optenv HUSKY_UST10_ENABLED 0)" />
   <xacro:arg name="laser_ust10_front_prefix"  default="$(optenv HUSKY_UST10_PREFIX front)" />
   <xacro:arg name="laser_ust10_front_parent"  default="$(optenv HUSKY_UST10_PARENT top_plate_link)" />
@@ -15,5 +15,5 @@
   <xacro:arg name="laser_ust10_front_xyz"     default="$(optenv HUSKY_UST10_XYZ 0.2206 0.0 0.00635)" />
   <xacro:arg name="laser_ust10_front_rpy"     default="$(optenv HUSKY_UST10_RPY 0 0 0)" />
-  <xacro:arg name="laser_ust10_rear_enabled"  default="false" />
+  <xacro:arg name="laser_ust10_rear_enabled"  default="$(optenv HUSKY_UST10_SECONDARY_ENABLED 0)" />
   <xacro:arg name="laser_ust10_rear_prefix"   default="$(optenv HUSKY_UST10_SECONDARY_PREFIX rear)" />
   <xacro:arg name="laser_ust10_rear_parent"   default="$(optenv HUSKY_UST10_SECONDARY_PARENT top_plate_link)" />
@@ -21,5 +21,5 @@
   <xacro:arg name="laser_ust10_rear_xyz"      default="$(optenv HUSKY_UST10_SECONDARY_XYZ -0.2206 0.0 0.00635)" />
   <xacro:arg name="laser_ust10_rear_rpy"      default="$(optenv HUSKY_UST10_SECONDARY_RPY 0 0 3.14159)" />
-  <xacro:arg name="laser_3d_enabled" default="false" />
+  <xacro:arg name="laser_3d_enabled" default="$(optenv HUSKY_LASER_3D_ENABLED 0)" />
   <xacro:arg name="laser_3d_xyz" default="$(optenv HUSKY_LASER_3D_XYZ 0 0 0)" />
   <xacro:arg name="laser_3d_rpy" default="$(optenv HUSKY_LASER_3D_RPY 0 0 0)" />
@@ -29,5 +29,5 @@
   <xacro:arg name="realsense_mount" default="$(optenv HUSKY_REALSENSE_MOUNT_FRAME sensor_arch_mount_link)" />
   <!-- Custom addition to xacro file to include ZED2 camera ; by Dev Vaibhav-->
-  <xacro:arg name="zed2_enabled" default="$(optenv HUSKY_ZED2_ENABLED false)" />
+  <xacro:arg name="zed2_enabled" default="$(optenv HUSKY_ZED2_ENABLED 0)" />
   <xacro:arg name="zed2_xyz" default="$(optenv HUSKY_ZED2_XYZ 0 0.14 0)" />
   <xacro:arg name="zed2_rpy" default="$(optenv HUSKY_ZED2_RPY 0 0 0)" />
@@ -173,5 +173,5 @@
   <xacro:if value="$(arg sensor_arch)">
     <xacro:sensor_arch prefix="" parent="top_plate_link" size="$(arg sensor_arch_height)">
-        <origin xyz="$(optenv HUSKY_SENSOR_ARCH_OFFSET 0 0 0.5)" rpy="$(optenv HUSKY_SENSOR_ARCH_RPY 0 0 0)"/>
+        <origin xyz="$(optenv HUSKY_SENSOR_ARCH_OFFSET 0 0 0)" rpy="$(optenv HUSKY_SENSOR_ARCH_RPY 0 0 0)"/>
     </xacro:sensor_arch>
   </xacro:if>
@@ -186,5 +186,5 @@
       <xacro:intel_realsense_mount prefix="camera" topic="realsense" parent_link="realsense_mountpoint"/>
     </xacro:if>
-  <!-- Custom addition to xacro file to include ZED2 camera ; by Dev Vaibhav-->
+    <!-- Custom addition to xacro file to include ZED2 camera ; by Dev Vaibhav-->
   <!-- add the zed2 to the sensor arch if needed -->
   <xacro:if value="$(arg zed2_enabled)">
@@ -195,4 +195,282 @@
       <child link="zed2_mountpoint" />
     </joint>
+      <!-- Camera Center -->
+      <link name="zed2_camera_center">
+        <inertial>
+          <mass value="0.16140"/>
+          <origin xyz="0 0 0"/>
+          <inertia
+            ixx="0.0003947" ixy="0.0" ixz="3.3365e-8"
+            iyy="2.417e-5" iyz="0.0"
+            izz="0.0003973"/>
+        </inertial>
+        <visual>
+          <geometry>
+            <mesh filename="package://husky_description/meshes/accessories/ZED2.dae"/>
+          </geometry>
+        </visual>
+        <collision>
+          <geometry>
+            <mesh filename="package://husky_description/meshes/accessories/ZED2.dae"/>
+          </geometry>
+        </collision>
+      </link>
+      <!-- Custom addition to xacro file to include ZED2 camera ; by Dev Vaibhav-->
+      <joint name="zed2_camera_center_joint" type="fixed">
+        <parent link="zed2_mountpoint"/>
+        <child link="zed2_camera_center"/>
+        <origin xyz="0 0 0" rpy="0 0 0" />
+      </joint>
+      <!-- Left Camera -->
+      <joint name="zed2_left_camera_joint" type="fixed">
+        <parent link="zed2_camera_center"/>
+        <child link="zed2_left_camera_frame"/>
+        <origin xyz="0 0.06 0" rpy="0 0 0" />
+      </joint>
+      <link name="zed2_left_camera_frame" />
+      <joint name="zed2_left_camera_optical_joint" type="fixed">
+        <origin xyz="0 0 0" rpy="-${pi/2} 0.0 -${pi/2}"/>
+        <parent link="zed2_left_camera_frame"/>
+        <child link="zed2_left_camera_optical_frame"/>
+      </joint>
+      <link name="zed2_left_camera_optical_frame"/>
+      <!-- Right Camera -->
+      <joint name="zed2_right_camera_joint" type="fixed">
+        <parent link="zed2_camera_center"/>
+        <child link="zed2_right_camera_frame"/>
+        <origin xyz="0 -0.06 0" rpy="0 0 0" />
+      </joint>
+      <link name="zed2_right_camera_frame" />
+      <joint name="zed2_right_camera_optical_joint" type="fixed">
+        <origin xyz="0 0 0" rpy="-${pi/2} 0.0 -${pi/2}"/>
+        <parent link="zed2_right_camera_frame"/>
+        <child link="zed2_right_camera_optical_frame"/>
+      </joint>
+      <link name="zed2_right_camera_optical_frame"/>
+      <!-- Sensors -->
+      <joint name="zed2_mag_joint" type="fixed">
+        <parent link="zed2_camera_center"/>
+        <child link="zed2_mag_link"/>
+        <origin xyz="0 0 0" rpy="0 0 0" />
+      </joint>
+      <link name="zed2_mag_link" />
+      <joint name="zed2_baro_joint" type="fixed">
+        <parent link="zed2_camera_center"/>
+        <child link="zed2_baro_link"/>
+        <origin xyz="0 0 0" rpy="0 0 0" />
+      </joint>
+      <link name="zed2_baro_link" />
+      <joint name="zed2_temp_left_joint" type="fixed">
+        <parent link="zed2_left_camera_frame"/>
+        <child link="zed2_temp_left_link"/>
+        <origin xyz="0 0 0" rpy="0 0 0" />
+      </joint>
+      <link name="zed2_temp_left_link" />
+      <joint name="zed2_temp_right_joint" type="fixed">
+          <parent link="zed2_right_camera_frame"/>
+          <child link="zed2_temp_right_link"/>
+          <origin xyz="0 0 0" rpy="0 0 0" />
+      </joint>
+      <link name="zed2_temp_right_link" />
+      <!-- Left/Depth camera -->
+      <gazebo reference="zed2_left_camera_frame">
+        <!-- Raw images (with lens distortion) -->
+        <sensor type="camera" name="zed2_left_raw_camera">
+          <always_on>true</always_on>
+          <update_rate>15.0</update_rate>
+          <visualize>false</visualize>
+          <camera name="zed2_left_raw">
+            <horizontal_fov>1.7633</horizontal_fov>
+            <image>
+              <width>1280</width>
+              <height>720</height>
+              <format>R8G8B8</format>
+            </image>
+            <clip>
+              <near>0.02</near>
+              <far>300</far>
+            </clip>
+            <noise>
+              <type>gaussian</type>
+              <mean>0.0</mean>
+              <stddev>0.007</stddev>
+            </noise>
+            <distortion>
+              <!-- Values copied from an actual ZED2 camera -->
+              <k1>-0.043693598</k1>
+              <k2>0.0146164996</k2>
+              <p1>-0.006573319</p1>
+              <p2>-0.000216900</p2>
+              <k3>0.000084328</k3>
+              <center>0.5 0.5</center>
+            </distortion>
+          </camera>
+          <plugin name="camera_controller" filename="libgazebo_ros_camera.so">
+            <robotNamespace>/</robotNamespace>
+            <cameraName>zed2/left_raw</cameraName>
+            <imageTopicName>image_raw_color</imageTopicName>
+            <cameraInfoTopicName>camera_info</cameraInfoTopicName>
+            <frameName>zed2_left_camera_optical_frame</frameName>
+            <distortionK1>-0.043693598</distortionK1>
+            <distortionK2>0.0146164996</distortionK2>
+            <distortionT1>-0.006573319</distortionT1>
+            <distortionT2>-0.000216900</distortionT2>
+            <distortionK3>0.000084328</distortionK3>
+            <CxPrime>648.5</CxPrime>
+            <Cx>648.5</Cx>
+            <Cy>366.8340148925781</Cy>
+            <hackBaseline>0.0</hackBaseline>
+          </plugin>
+        </sensor>
+        <sensor type="depth" name="zed2_left_camera">
+          <!-- Rectified images, Depth images, Point Clouds -->
+          <always_on>true</always_on>
+          <update_rate>15.0</update_rate>
+          <visualize>false</visualize>
+          <camera name="zed2_left">
+            <horizontal_fov>1.7633</horizontal_fov>
+            <image>
+              <width>1280</width>
+              <height>720</height>
+              <format>R8G8B8</format>
+            </image>
+            <clip>
+              <near>0.02</near>
+              <far>300</far>
+            </clip>
+            <noise>
+              <type>gaussian</type>
+              <mean>0.0</mean>
+              <stddev>0.007</stddev>
+            </noise>
+          </camera>
+          <plugin name="camera_controller" filename="libgazebo_ros_openni_kinect.so">
+            <robotNamespace>/</robotNamespace>
+            <cameraName>zed2</cameraName>
+            <imageTopicName>left/image_rect_color</imageTopicName>
+            <cameraInfoTopicName>left/camera_info</cameraInfoTopicName>
+            <depthImageTopicName>depth/depth_registered</depthImageTopicName>
+            <depthImageInfoTopicName>depth/camera_info</depthImageInfoTopicName>
+            <pointCloudTopicName>point_cloud/cloud_registered</pointCloudTopicName>
+            <pointCloudCutoff>0.3</pointCloudCutoff>
+            <pointCloudCutoffMax>20.0</pointCloudCutoffMax>
+            <frameName>zed2_left_camera_optical_frame</frameName>
+            <baseline>0.12</baseline>
+            <CxPrime>658.8206787109375</CxPrime>
+            <Cx>658.8206787109375</Cx>
+            <Cy>372.25787353515625</Cy>
+            <hackBaseline>0.0</hackBaseline>
+          </plugin>
+        </sensor>
+      </gazebo>
+      <!-- Right camera -->
+      <gazebo reference="zed2_right_camera_frame">
+        <!-- Raw images (with lens distortion) -->
+        <sensor type="camera" name="zed2_right_raw_camera">
+          <always_on>true</always_on>
+          <update_rate>15.0</update_rate>
+          <visualize>false</visualize>
+          <camera name="zed2_right_raw">
+            <horizontal_fov>1.7633</horizontal_fov>
+            <image>
+              <width>1280</width>
+              <height>720</height>
+              <format>R8G8B8</format>
+            </image>
+            <clip>
+              <near>0.02</near>
+              <far>300</far>
+            </clip>
+            <noise>
+              <type>gaussian</type>
+              <mean>0.0</mean>
+              <stddev>0.007</stddev>
+            </noise>
+            <distortion>
+              <k1>-0.040993299</k1>
+              <k2>0.009593590</k2>
+              <p1>-0.004429849</p1>
+              <p2>0.000192024</p2>
+              <k3>-0.000320880</k3>
+              <center>0.5 0.5</center>
+            </distortion>
+          </camera>
+          <plugin name="camera_controller" filename="libgazebo_ros_camera.so">
+            <robotNamespace>/</robotNamespace>
+            <cameraName>zed2/right_raw</cameraName>
+            <imageTopicName>image_raw_color</imageTopicName>
+            <cameraInfoTopicName>camera_info</cameraInfoTopicName>
+            <frameName>zed2_right_camera_optical_frame</frameName>
+            <distortionK1>-0.040993299</distortionK1>
+            <distortionK2>0.009593590</distortionK2>
+            <distortionT1>-0.004429849</distortionT1>
+            <distortionT2>0.000192024</distortionT2>
+            <distortionK3>-0.000320880</distortionK3>
+            <CxPrime>659.3049926757812</CxPrime>
+            <Cx>659.3049926757812</Cx>
+            <Cy>371.39849853515625</Cy>
+            <hackBaseline>0.12</hackBaseline>
+          </plugin>
+        </sensor>
+        <sensor type="camera" name="zed2_right_camera">
+          <!-- Rectified images -->
+          <always_on>true</always_on>
+          <update_rate>15.0</update_rate>
+          <visualize>false</visualize>
+          <camera name="zed2_right">
+            <horizontal_fov>1.7633</horizontal_fov>
+            <image>
+              <width>1280</width>
+              <height>720</height>
+              <format>R8G8B8</format>
+            </image>
+            <clip>
+              <near>0.02</near>
+              <far>300</far>
+            </clip>
+            <noise>
+              <type>gaussian</type>
+              <mean>0.0</mean>
+              <stddev>0.007</stddev>
+            </noise>
+          </camera>
+          <plugin name="camera_controller" filename="libgazebo_ros_camera.so">
+            <robotNamespace>/</robotNamespace>
+            <cameraName>zed2/right</cameraName>
+            <imageTopicName>image_rect_color</imageTopicName>
+            <cameraInfoTopicName>camera_info</cameraInfoTopicName>
+            <frameName>zed2_right_camera_optical_frame</frameName>
+            <CxPrime>658.8206787109375</CxPrime>
+            <Cx>658.8206787109375</Cx>
+            <Cy>372.25787353515625</Cy>
+            <hackBaseline>0.12</hackBaseline>
+          </plugin>
+        </sensor>
+      </gazebo>
+      <!-- IMU -->
+      <gazebo reference="zed2_left_camera_frame">
+        <sensor type="imu" name="zed2_imu_sensor">
+          <update_rate>100</update_rate>
+          <plugin filename="libgazebo_ros_imu_sensor.so" name="imu_plugin">
+            <robotNamespace>/</robotNamespace>
+            <topicName>zed2/imu/data</topicName>
+            <frameName>zed2_imu_link</frameName>
+            <updateRateHZ>100.0</updateRateHZ>
+            <gaussianNoise>0.01</gaussianNoise>
+            <initialOrientationAsReference>false</initialOrientationAsReference>
+            <!-- IMU frame offset copied from an actual ZED2 camera -->
+            <xyzOffset>-0.002 -0.023 -0.002</xyzOffset>
+            <rpyOffset>0.0014025 -0.0000012 -0.0016915</rpyOffset>
+          </plugin>
+        </sensor>
+      </gazebo>
+  </xacro:if>
+  <!--
+    Add the 3d laser to the sensor arch if needed
+  -->
+  <xacro:if value="$(arg laser_3d_enabled)">
+    <xacro:vlp16_mount prefix="" parent_link="sensor_arch_mount_link" topic="$(optenv HUSKY_LASER_3D_TOPIC points)">
+      <origin xyz="$(arg laser_3d_xyz)" rpy="$(arg laser_3d_rpy)" />
+    </xacro:vlp16_mount>
   </xacro:if>
     <ros2_control name="${prefix}husky_hardware" type="system">
