Commit message: implemented zed2

File: install/husky_description/share/husky_description/urdf/accessories/sensor_arch.urdf.xacro (robot description, xacro)
@@ -3,5 +3,5 @@
   <xacro:macro name="sensor_arch" params="prefix parent size:=510 *origin">
       <!-- Robot Base -->
-      <!--xacro:macro name="box_inertia" params="m w h d">
+      <xacro:macro name="box_inertia" params="m w h d">
         <inertial>
           <origin xyz="0 0 0" rpy="0 0 0"/>
@@ -9,32 +9,25 @@
           <inertia ixx="${(m/12) * (h*h + d*d)}" ixy="0.0" ixz="0.0" iyy="${(m/12) * (w*w + d*d)}" iyz="0.0" izz="${(m/12) * (w*w + h*h)}"/>
         </inertial>
-      </xacro:macro>-->
-  <link name="${prefix}sensor_arch_base_link" />
+      </xacro:macro>
   <link name="${prefix}sensor_arch_mount_link">
      <origin xyz="0 0 0" rpy="0 0 0"/>
      <visual>
-	<geometry>
+	    <geometry>
 	     <mesh filename="file://$(find husky_description)/meshes/accessories/${510}_mm_sensor_arch.dae" />
-        </geometry>
-    </visual>
+      </geometry>
+     </visual>
     <collision>
-	<origin xyz="0 0 0" rpy="0 0 0"/>
-	<geometry>
+	    <origin xyz="0 0 0" rpy="0 0 0"/>
+	    <geometry>
 	     <mesh filename="file://$(find husky_description)/meshes/accessories/${510}_mm_sensor_arch.dae" />
-        </geometry>
+      </geometry>
     </collision>
-    <!--<xacro:box_inertia m=".01" w=".01" d=".01" h=".01"/>-->
+    <xacro:box_inertia m=".01" w=".01" d=".01" h=".01"/>
   </link>
-  <joint name="${prefix}sensor_arch_base_link_joint" type="fixed">
+  <joint name="${prefix}sensor_arch_mount" type="fixed">
+  	    <xacro:insert_block name="origin" />
             <parent link="${parent}" />
-            <child link="${prefix}sensor_arch_base_link" />
-            <xacro:insert_block name="origin" />
-        </joint>
-        <!-- Attach the sensor arch to the top plate -->
-        <joint name="${prefix}sensor_arch_mount" type="fixed">
-             <parent link="${prefix}sensor_arch_base_link"/>
-             <child link="${prefix}sensor_arch_mount_link"/>
-             <origin xyz="0 0 ${size/1000}" rpy="0 0 0" />
-        </joint>
+            <child link="${prefix}sensor_arch_mount_link" />
+  </joint>
 </xacro:macro>
 </robot>

File: install/husky_description/share/husky_description/urdf/husky_macro.urdf.xacro (robot description, xacro)
@@ -24,10 +24,10 @@
   <xacro:arg name="laser_3d_xyz" default="$(optenv HUSKY_LASER_3D_XYZ 0 0 0)" />
   <xacro:arg name="laser_3d_rpy" default="$(optenv HUSKY_LASER_3D_RPY 0 0 0)" />
-  <xacro:arg name="realsense_enabled" default="$(optenv HUSKY_REALSENSE_ENABLED 1)" />
+  <xacro:arg name="realsense_enabled" default="$(optenv HUSKY_REALSENSE_ENABLED 0)" />
   <xacro:arg name="realsense_xyz" default="$(optenv HUSKY_REALSENSE_XYZ 0 0 0)" />
   <xacro:arg name="realsense_rpy" default="$(optenv HUSKY_REALSENSE_RPY 0 0 0)" />
   <xacro:arg name="realsense_mount" default="$(optenv HUSKY_REALSENSE_MOUNT_FRAME sensor_arch_mount_link)" />
   <!-- Custom addition to xacro file to include ZED2 camera ; by Dev Vaibhav-->
-  <xacro:arg name="zed2_enabled" default="$(optenv HUSKY_ZED2_ENABLED 0)" />
+  <xacro:arg name="zed2_enabled" default="$(optenv HUSKY_ZED2_ENABLED 1)" />
   <xacro:arg name="zed2_xyz" default="$(optenv HUSKY_ZED2_XYZ 0 0.14 0)" />
   <xacro:arg name="zed2_rpy" default="$(optenv HUSKY_ZED2_RPY 0 0 0)" />
@@ -173,5 +173,5 @@
   <xacro:if value="$(arg sensor_arch)">
     <xacro:sensor_arch prefix="" parent="top_plate_link" size="$(arg sensor_arch_height)">
-        <origin xyz="$(optenv HUSKY_SENSOR_ARCH_OFFSET 0 0 0)" rpy="$(optenv HUSKY_SENSOR_ARCH_RPY 0 0 0)"/>
+        <origin xyz="$(optenv HUSKY_SENSOR_ARCH_OFFSET 0 0 0.5)" rpy="$(optenv HUSKY_SENSOR_ARCH_RPY 0 0 0)"/>
     </xacro:sensor_arch>
   </xacro:if>
@@ -186,5 +186,5 @@
       <xacro:intel_realsense_mount prefix="camera" topic="realsense" parent_link="realsense_mountpoint"/>
     </xacro:if>
-    <!-- Custom addition to xacro file to include ZED2 camera ; by Dev Vaibhav-->
+  <!-- Custom addition to xacro file to include ZED2 camera ; by Dev Vaibhav-->
   <!-- add the zed2 to the sensor arch if needed -->
   <xacro:if value="$(arg zed2_enabled)">
@@ -207,10 +207,10 @@
         <visual>
           <geometry>
-            <mesh filename="package://husky_description/meshes/accessories/ZED2.dae"/>
+            <mesh filename="file://$(find husky_description)/meshes/accessories/ZED2.dae"/>
           </geometry>
         </visual>
         <collision>
           <geometry>
-            <mesh filename="package://husky_description/meshes/accessories/ZED2.dae"/>
+            <mesh filename="file://$(find husky_description)/meshes/accessories/ZED2.dae"/>
           </geometry>
         </collision>
