Commit message: Added VLP 3D laser

File: install/husky_description/share/husky_description/urdf/accessories/vlp16_mount.urdf.xacro (robot description, xacro)
@@ -1,9 +1,6 @@
 <?xml version="1.0"?>
 <robot xmlns:xacro="http://wiki.ros.org/xacro">
-  <xacro:include filename="$(find velodyne_description)/urdf/VLP-16.urdf.xacro" />
-  <xacro:macro name="vlp16_mount" params="prefix parent_link topic height:=0.12 *origin">
-    <!--
-      The VLP16 is mounted to a pair of extrusion rods on top of the main sensor arch
-    -->
+<xacro:include filename="$(find husky_description)/urdf/accessories/VLP-16.urdf.xacro"/>
+  <xacro:macro name="laser_vlp16_mount" params="prefix parent_link topic height:=0.12">
     <link name="${prefix}vlp16_mount_base_link" />
     <link name="${prefix}vlp16_mount_plate">
@@ -41,5 +38,5 @@
       </collision>
     </link>
-    <link name="${prefix}vlp16_mount_right_support">
+     <link name="${prefix}vlp16_mount_right_support">
       <visual>
         <geometry>
@@ -61,5 +58,4 @@
       <parent link="${parent_link}" />
       <child link="${prefix}vlp16_mount_base_link" />
-      <xacro:insert_block name="origin" />
     </joint>
     <joint name="${prefix}vlp16_mount_left_support_joint" type="fixed">
@@ -81,4 +77,4 @@
       <origin xyz="0 0 0.0063" rpy="0 0 0" />
     </xacro:VLP-16>
-  </xacro:macro>
+    </xacro:macro>
 </robot>

File: install/husky_description/share/husky_description/urdf/husky_macro.urdf.xacro (robot description, xacro)
@@ -1,12 +1,4 @@
 <?xml version="1.0"?>
 <robot name="husky" xmlns:xacro="http://ros.org/wiki/xacro">
-  <!-- lms1xx_xyz broken - but I don't think we're using this.
-  <xacro:arg name="laser_enabled" default="$(optenv HUSKY_LMS1XX_ENABLED 0)" />
-  <xacro:arg name="laser_xyz" default="$(optenv HUSKY_LMS1XX_XYZ 0.2206 0.0 0.00635)" />
-  <xacro:arg name="laser_rpy" default="$(optenv HUSKY_LMS1XX_RPY 0.0 0.0 0.0)" />
-  <xacro:arg name="laser_secondary_enabled" default="$(optenv HUSKY_LMS1XX_SECONDARY_ENABLED 0)" />
-  <xacro:arg name="laser_secondary_xyz" default="$(optenv HUSKY_LMS1XX_SECONDARY_XYZ -0.2206 0.0 0.00635)" />
-  <xacro:arg name="laser_secondary_rpy" default="$(optenv HUSKY_LMS1XX_SECONDARY_RPY 0.0 0.0 3.14159)" />
--->
   <xacro:arg name="laser_ust10_front_enabled" default="$(optenv HUSKY_UST10_ENABLED 1)" />
   <xacro:arg name="laser_ust10_front_prefix"  default="$(optenv HUSKY_UST10_PREFIX front)" />
@@ -21,8 +13,9 @@
   <xacro:arg name="laser_ust10_rear_xyz"      default="$(optenv HUSKY_UST10_SECONDARY_XYZ -0.2206 0.0 0.00635)" />
   <xacro:arg name="laser_ust10_rear_rpy"      default="$(optenv HUSKY_UST10_SECONDARY_RPY 0 0 3.14159)" />
-  <xacro:arg name="laser_3d_enabled" default="$(optenv HUSKY_LASER_3D_ENABLED 0)" />
+  <xacro:arg name="laser_3d_enabled" default="$(optenv HUSKY_LASER_3D_ENABLED 1)" />
   <xacro:arg name="laser_3d_xyz" default="$(optenv HUSKY_LASER_3D_XYZ 0 0 0)" />
   <xacro:arg name="laser_3d_rpy" default="$(optenv HUSKY_LASER_3D_RPY 0 0 0)" />
-  <xacro:arg name="realsense_enabled" default="$(optenv HUSKY_REALSENSE_ENABLED 0)" />
+  <xacro:arg name="laser_3d_mount" default="$(optenv HUSKY_LASER_3D_MOUNT_FRAME sensor_arch_mount_link)" />
+  <xacro:arg name="realsense_enabled" default="$(optenv HUSKY_REALSENSE_ENABLED 1)" />
   <xacro:arg name="realsense_xyz" default="$(optenv HUSKY_REALSENSE_XYZ 0 0 0)" />
   <xacro:arg name="realsense_rpy" default="$(optenv HUSKY_REALSENSE_RPY 0 0 0)" />
@@ -49,7 +42,6 @@
   <xacro:include filename="$(find husky_description)/urdf/accessories/intel_realsense.urdf.xacro" />
   <xacro:include filename="$(find husky_description)/urdf/accessories/hokuyo_ust10.urdf.xacro" />
-  <!--<xacro:include filename="$(find husky_description)/urdf/accessories/sick_lms1xx_mount.urdf.xacro" />
   <xacro:include filename="$(find husky_description)/urdf/accessories/vlp16_mount.urdf.xacro"/>
-  -->
+  <xacro:include filename="$(find husky_description)/urdf/accessories/VLP-16.urdf.xacro"/>
   <xacro:include filename="$(find husky_description)/urdf/accessories/sensor_arch.urdf.xacro"/>
   <xacro:include filename="$(find husky_description)/urdf/accessories/zed2.xacro"/>
@@ -186,4 +178,16 @@
       <xacro:intel_realsense_mount prefix="camera" topic="realsense" parent_link="realsense_mountpoint"/>
     </xacro:if>
+    <!--
+    Add the 3d laser to the sensor arch if needed
+  -->
+  <xacro:if value="$(arg laser_3d_enabled)">
+    <link name="laser_3d_mountpoint"/>
+    <joint name="laser_3d_mountpoint_joint" type="fixed">
+      <origin xyz="0 0 0" rpy="0 0 0" />
+      <parent link="$(arg laser_3d_mount)"/>
+      <child link="laser_3d_mountpoint" />
+    </joint>
+    <xacro:laser_vlp16_mount prefix="" parent_link="realsense_mountpoint" topic="points"/>
+  </xacro:if>
   <!-- Custom addition to xacro file to include ZED2 camera ; by Dev Vaibhav-->
   <!-- add the zed2 to the sensor arch if needed -->
@@ -466,12 +470,4 @@
       </gazebo>
   </xacro:if>
-  <!--
-    Add the 3d laser to the sensor arch if needed
-  -->
-  <xacro:if value="$(arg laser_3d_enabled)">
-    <xacro:vlp16_mount prefix="" parent_link="sensor_arch_mount_link" topic="$(optenv HUSKY_LASER_3D_TOPIC points)">
-      <origin xyz="$(arg laser_3d_xyz)" rpy="$(arg laser_3d_rpy)" />
-    </xacro:vlp16_mount>
-  </xacro:if>
     <ros2_control name="${prefix}husky_hardware" type="system">
       <hardware>

File: src/husky/husky_description/urdf/accessories/vlp16_mount.urdf (copy).xacro (robot description, xacro)
@@ -1,6 +1,9 @@
 <?xml version="1.0"?>
 <robot xmlns:xacro="http://wiki.ros.org/xacro">
-<xacro:include filename="$(find husky_description)/urdf/accessories/VLP-16.urdf.xacro"/>
-  <xacro:macro name="laser_vlp16_mount" params="prefix parent_link topic height:=0.12">
+ <xacro:include filename="$(find husky_description)/urdf/accessories/VLP-16.urdf.xacro"/>
+  <xacro:macro name="vlp_laser_3d_mount" params="prefix parent_link topic height:=0.12 *origin">
+    <!--
+      The VLP16 is mounted to a pair of extrusion rods on top of the main sensor arch
+    -->
     <link name="${prefix}vlp16_mount_base_link" />
     <link name="${prefix}vlp16_mount_plate">
@@ -38,5 +41,5 @@
       </collision>
     </link>
-     <link name="${prefix}vlp16_mount_right_support">
+    <link name="${prefix}vlp16_mount_right_support">
       <visual>
         <geometry>
@@ -58,4 +61,5 @@
       <parent link="${parent_link}" />
       <child link="${prefix}vlp16_mount_base_link" />
+      <xacro:insert_block name="origin" />
     </joint>
     <joint name="${prefix}vlp16_mount_left_support_joint" type="fixed">
@@ -77,4 +81,4 @@
       <origin xyz="0 0 0.0063" rpy="0 0 0" />
     </xacro:VLP-16>
-    </xacro:macro>
+  </xacro:macro>
 </robot>
